File: board/ICE40UP-Development-Board.kicad_sch (KiCad schematic)
At the start: 93 parts, among them Q1 Q_PJFET_GSD, X1 Conn_01x01, X10 Conn_01x01, X11 Conn_01x01, X12 Conn_01x01, X13 Conn_01x01, X14 Conn_01x01, X15 Conn_01x01, X16 Conn_01x01, X17 Conn_01x01, X18 Conn_01x01, X19 Conn_01x01, X2 Conn_01x01, X20 Conn_01x01, X21 Conn_01x01, X22 Conn_01x01, X23 Conn_01x01, X24 Conn_01x01, X25 Conn_01x01, X26 Conn_01x01, X3 Conn_01x01, X4 Conn_01x01, X5 USB4105-GF-A, X6 Conn_01x01, X7 Conn_01x01, X8 Conn_01x01, X9 Conn_01x01, Y1 48MHz

Commit message: add footprints
Parts:
- added X2, X3, X4: Conn_01x01, myLib:PinHeader_1x01_P2.54mm_Vertical, symbol Connector_Generic:Conn_01x01
- JP1, JP2: footprint Jumper:SolderJumper-2_P1.3mm_Open_Pad1.0x1.5mm -> Jumper:SolderJumper-2_P1.3mm_Open_RoundedPad1.0x1.5mm
- Q1: footprint (none) -> Package_TO_SOT_SMD:SOT-723
- R1: renamed from R5; footprint (none) -> Resistor_SMD:R_01005_0402Metric
- R10: footprint (none) -> Resistor_SMD:R_01005_0402Metric
- R11: renamed from R7; footprint (none) -> Resistor_SMD:R_01005_0402Metric
- R12: renamed from R13; footprint (none) -> Resistor_SMD:R_01005_0402Metric
- R13: renamed from R6; footprint (none) -> Resistor_SMD:R_01005_0402Metric
- R14: renamed from R9; footprint (none) -> Resistor_SMD:R_01005_0402Metric
- R2: renamed from R11; footprint (none) -> Resistor_SMD:R_01005_0402Metric
- R3: renamed from R8; footprint (none) -> Resistor_SMD:R_01005_0402Metric
- R4: renamed from R12; footprint (none) -> Resistor_SMD:R_01005_0402Metric
- R5: renamed from R2; footprint (none) -> Resistor_SMD:R_01005_0402Metric
- R6: renamed from R3; footprint (none) -> Resistor_SMD:R_01005_0402Metric
- R7: renamed from R1; footprint (none) -> Resistor_SMD:R_01005_0402Metric
- R8: renamed from R4; footprint (none) -> Resistor_SMD:R_01005_0402Metric
- R9: renamed from R14; footprint (none) -> Resistor_SMD:R_01005_0402Metric
- S1, S2: footprint (none) -> myLib:SW_SPST_EVQP2
- TP1: footprint (none) -> myLib:PinSocket_1x01_P2.54mm_Vertical_SMD
- TP10, TP11, TP12, TP2, TP3, TP4, TP5, TP6, TP7, TP8, TP9: footprint TestPoint:TestPoint_Pad_D1.0mm -> myLib:PinSocket_1x01_P2.54mm_Vertical_SMD
- V3: renamed from V9; footprint Package_SO:SOIC-8_5.23x5.23mm_P1.27mm -> Package_SON:SON-8-1EP_3x2mm_P0.5mm_EP1.4x1.6mm
- V5: renamed from V4; footprint Package_TO_SOT_SMD:SOT-23-5 -> Package_DFN_QFN:UDFN-4-1EP_1x1mm_P0.65mm_EP0.48x0.48mm
- V8: renamed from V7; footprint (none) -> myLib:CREE_UHD111A
- X1: renamed from X5; footprint (none) -> Connector_USB:USB_C_Receptacle_G-Switch_GT-USB-7010ASV
- X10: footprint (none) -> myLib:PinHeader_1x01_P2.54mm_Vertical
- X11: renamed from X20; footprint (none) -> myLib:PinHeader_1x01_P2.54mm_Vertical
- X12: renamed from X21; footprint (none) -> myLib:PinHeader_1x01_P2.54mm_Vertical
- X13: renamed from X22; footprint (none) -> myLib:PinHeader_1x01_P2.54mm_Vertical
- X14: renamed from X23; footprint (none) -> myLib:PinHeader_1x01_P2.54mm_Vertical
- X15: renamed from X24; footprint (none) -> myLib:PinHeader_1x01_P2.54mm_Vertical
- X16: renamed from X25; footprint (none) -> myLib:PinHeader_1x01_P2.54mm_Vertical
- X17: renamed from X26; footprint (none) -> myLib:PinHeader_1x01_P2.54mm_Vertical
- X18: renamed from X4; footprint (none) -> myLib:PinHeader_1x01_P2.54mm_Vertical
- X19: renamed from X7; footprint (none) -> myLib:PinHeader_1x01_P2.54mm_Vertical
- X20: renamed from X9; footprint (none) -> myLib:PinHeader_1x01_P2.54mm_Vertical
- X21: renamed from X11; footprint (none) -> myLib:PinHeader_1x01_P2.54mm_Vertical
- X22: renamed from X12; footprint (none) -> myLib:PinHeader_1x01_P2.54mm_Vertical
- X23: renamed from X13; footprint (none) -> myLib:PinHeader_1x01_P2.54mm_Vertical
- X24: renamed from X14; footprint (none) -> myLib:PinHeader_1x01_P2.54mm_Vertical
- X25: renamed from X15; footprint (none) -> myLib:PinHeader_1x01_P2.54mm_Vertical
- X26: renamed from X16; footprint (none) -> myLib:PinHeader_1x01_P2.54mm_Vertical
- X27: renamed from X17; footprint (none) -> myLib:PinHeader_1x01_P2.54mm_Vertical
- X28: renamed from X18; footprint (none) -> myLib:PinHeader_1x01_P2.54mm_Vertical
- X29: renamed from X19; footprint (none) -> myLib:PinHeader_1x01_P2.54mm_Vertical
- X5: renamed from X1; footprint (none) -> myLib:PinHeader_1x01_P2.54mm_Vertical
- X6: renamed from X2; footprint (none) -> myLib:PinHeader_1x01_P2.54mm_Vertical
- X7: renamed from X3; footprint (none) -> myLib:PinHeader_1x01_P2.54mm_Vertical
- X8: renamed from X6; footprint (none) -> myLib:PinHeader_1x01_P2.54mm_Vertical
- X9: renamed from X8; footprint (none) -> myLib:PinHeader_1x01_P2.54mm_Vertical
- Y1: footprint Oscillator:Oscillator_SMD_Abracon_ASE-4Pin_3.2x2.5mm -> Oscillator:Oscillator_SMD_SeikoEpson_SG8002CE-4Pin_3.2x2.5mm
- renumbered C16 to C1, C14 to C10, C5 to C13, C6 to C14, C7 to C16, C19 to C17, C8 to C18, C9 to C19, C13 to C2, C10 to C20, C1 to C21, C18 to C22, C2 to C23, C20 to C5, C22 to C6, C17 to C7, C21 to C8, C23 to C9, V3 to V1, V6 to V2, V1 to V4, V5 to V6, V2 to V7, V8 to V9
Connections:
- net +3V3: now also X2.1 (Pin_1)
- net GND: now also X4.1 (Pin_1)
- net RGB0: now also V8.3 (RK); no longer V8.1 (RK)
- net RGB2: now also V8.1 (BK); no longer V8.3 (BK)
- net VBUS: now also V1.4 (VIN), V5.4 (VIN), X3.1 (Pin_1); no longer V1.1 (VIN), V5.1 (VIN)
- net at C2.1, JP1.1 (A): now also V1.1 (VOUT); no longer V1.5 (VOUT)
- net at C10.1, JP2.1 (A): now also V5.1 (VOUT); no longer V5.5 (VOUT)
Other:
- note added: "300mA max"
- note added: "?"
- note added: "p-channel mosfet footprints led green 0603"
- note removed: "memory typical application choose led led series r rgb series r footprints led green 0603"
- moved on the sheet: TP10, TP11, TP12, TP6, TP7, TP8, TP9

Commit message: add pcb layout
Parts:
- removed R8: 22R, Resistor_SMD:R_01005_0402Metric, symbol Device:R_Small
- added R7: 22R, Resistor_SMD:R_01005_0402Metric, symbol Device:R_Small
- renumbered R7 to R8
Connections:
- net USBD+: now also V4.1 (I/O1), R7.1; no longer V4.6 (I/O4)
- net USB_P+: now also R7.2
Other:
- moved on the sheet: R8, V4

Commit message: change ldo regulator ic
Parts:
- removed C1, C10, C2, C7: 1u, Capacitor_SMD:C_0402_1005Metric, symbol Device:C_Small
- removed Q1: Q_PJFET_GSD, Package_TO_SOT_SMD:SOT-723, symbol Device:Q_PJFET_GSD
- removed TP1: VBUS, myLib:PinSocket_1x01_P2.54mm_Vertical_SMD, symbol Connector:TestPoint
- removed V1: MIC5504-1.2YM5, Package_DFN_QFN:UDFN-4-1EP_1x1mm_P0.65mm_EP0.48x0.48mm, symbol Regulator_Linear:MIC5504-1.2YM5
- removed V5: MIC5504-3.3YM5, Package_DFN_QFN:UDFN-4-1EP_1x1mm_P0.65mm_EP0.48x0.48mm, symbol Regulator_Linear:MIC5504-3.3YM5
- added C11: 10u, Capacitor_SMD:C_0402_1005Metric, symbol Device:C_Small
- added C12, C16, C17: 1u, Capacitor_SMD:C_0402_1005Metric, symbol Device:C_Small
- added R7: 10k, Resistor_SMD:R_01005_0402Metric, symbol Device:R_Small
- added TP1: VBUS, myLib:PinSocket_1x01_P2.54mm_Vertical_SMD, symbol Connector:TestPoint_Small
- added V3: TLV7111233DSER, Package_SON:WSON-6_1.5x1.5mm_P0.5mm, symbol Regulator_Linear:MIC5355-S4YMME
- renumbered C21 to C1, C20 to C10, C11 to C13, C12 to C14, C22 to C18, C17 to C19, C23 to C2, C5 to C20, C8 to C21, C6 to C22, C9 to C23, C13 to C5, C14 to C6, C16 to C7, C18 to C8, C19 to C9, R7 to R1, R14 to R10, R10 to R11, R2 to R12, R4 to R13, R12 to R14, R9 to R15, R8 to R2, R5 to R3, R6 to R4, R1 to R5, R13 to R6, R11 to R8, R3 to R9, V7 to V1, V4 to V2, V6 to V4, V2 to V5, V8 to V6, V9 to V7, V3 to V8, V10 to V9, X2 to X1, X19 to X10, X9 to X11, X20 to X12, X10 to X13, X21 to X14, X22 to X15, X23 to X16, X24 to X17, X25 to X18, X26 to X19, X3 to X2, X27 to X20, X28 to X21, X29 to X22, X11 to X23, X12 to X24, X13 to X25, X14 to X26, X15 to X27, X16 to X28, X17 to X29, X4 to X3, X5 to X4, X6 to X5, X7 to X6, X18 to X7, X1 to X8, X8 to X9
Connections:
- net +1V2: now also JP1.1 (A), R7.2, V3.3 (NC); no longer JP1.2 (B)
- net +3V3: now also JP2.1 (A); no longer JP2.2 (B)
- net GND: now also C11.2, C12.2, C16.2, C17.2, R7.1, V3.4 (GND), V3.9 (GND)
- net VBUS: now also C11.1, C12.1, TP1.1, V3.1 (EN1), V3.2 (VIN)
- new net: C16.1, JP1.2 (B), V3.6 (VOUT1)
- new net: C17.1, JP2.2 (B), V3.5 (VOUT2)
Other:
- note added: "each 200mA max"
- note removed: "300mA max"
- note removed: "?"
- note removed: "D"
- note removed: "G"
- note removed: "S"
- note removed: "p-channel mosfet footprints led green 0603"
- moved on the sheet: C13, C14, JP1, JP2, R6

Commit message: finish schematic design
Parts:
- removed C19: 15p?, Capacitor_SMD:C_0402_1005Metric, symbol Device:C_Small
- removed R2: 22R, Resistor_SMD:R_01005_0402Metric, symbol Device:R_Small
- removed TP1: VBUS, myLib:PinSocket_1x01_P2.54mm_Vertical_SMD, symbol Connector:TestPoint_Small
- removed TP10, TP11, TP12, TP2, TP3, TP4, TP5, TP6, TP7, TP8, TP9: TestPoint_Small, myLib:PinSocket_1x01_P2.54mm_Vertical_SMD, symbol Connector:TestPoint_Small
- removed V2: USBLC6-4SC6, Package_TO_SOT_SMD:SOT-23-6, symbol Power_Protection:USBLC6-4SC6
- removed X1, X10, X11, X12, X13, X14, X15, X16, X17, X18, X19, X2, X20, X21, X22, X23, X24, X25, X26, X27, X28, X29, X3, X4, X5, X6, X7, X9: Conn_01x01, myLib:PinHeader_1x01_P2.54mm_Vertical, symbol Connector_Generic:Conn_01x01
- added R1: 1k5, Resistor_SMD:R_0402_1005Metric, symbol Device:R_Small
- added R11, R12, R13: 100R, Resistor_SMD:R_0402_1005Metric, symbol Device:R_Small
- added R5: 22R, Resistor_SMD:R_0402_1005Metric, symbol Device:R_Small
- added V2: USBLC6-2P6, Package_TO_SOT_SMD:SOT-666, symbol Power_Protection:USBLC6-2P6
- added X2, X3: Conn_01x16, Connector_PinHeader_2.54mm:PinHeader_1x16_P2.54mm_Vertical, symbol Connector_Generic:Conn_01x16
- added X4: Tag-Connect, Connector:Tag-Connect_TC2050-IDC-NL_2x05_P1.27mm_Vertical, symbol Connector_Generic:Conn_01x10
- R10: renamed from R9; footprint Resistor_SMD:R_01005_0402Metric -> Resistor_SMD:R_0402_1005Metric
- R14: renamed from R10; footprint Resistor_SMD:R_01005_0402Metric -> Resistor_SMD:R_0402_1005Metric
- R15: renamed from R11; footprint Resistor_SMD:R_01005_0402Metric -> Resistor_SMD:R_0402_1005Metric
- R16: renamed from R12; footprint Resistor_SMD:R_01005_0402Metric -> Resistor_SMD:R_0402_1005Metric
- R17: renamed from R13; footprint Resistor_SMD:R_01005_0402Metric -> Resistor_SMD:R_0402_1005Metric
- R18: renamed from R14; footprint Resistor_SMD:R_01005_0402Metric -> Resistor_SMD:R_0402_1005Metric
- R19: renamed from R15; footprint Resistor_SMD:R_01005_0402Metric -> Resistor_SMD:R_0402_1005Metric
- R2: renamed from R1; footprint Resistor_SMD:R_01005_0402Metric -> Resistor_SMD:R_0402_1005Metric
- R3, R4, R7: footprint Resistor_SMD:R_01005_0402Metric -> Resistor_SMD:R_0402_1005Metric
- R6: renamed from R5; footprint Resistor_SMD:R_01005_0402Metric -> Resistor_SMD:R_0402_1005Metric
- R8: renamed from R6; footprint Resistor_SMD:R_01005_0402Metric -> Resistor_SMD:R_0402_1005Metric
- R9: renamed from R8; footprint Resistor_SMD:R_01005_0402Metric -> Resistor_SMD:R_0402_1005Metric
- Y1: footprint Oscillator:Oscillator_SMD_SeikoEpson_SG8002CE-4Pin_3.2x2.5mm -> Oscillator:Oscillator_SMD_Abracon_ASE-4Pin_3.2x2.5mm
- renumbered C16 to C13, C17 to C14, C13 to C16, C14 to C17, C20 to C19, C21 to C20, C22 to C21, C23 to C22, X8 to X1
Connections:
- net +1V2: now also C5.2, C6.2, C7.2, X2.2 (Pin_2)
- net +3V3: now also X2.1 (Pin_1); no longer C5.2, C6.2, C7.2
- net CLK: now also V1.12 (IOB_22b)
- net FLASH_~{SS}: now also X3.16 (Pin_16), X4.10 (Pin_10)
- net GND: now also V2.2 (GND), X2.16 (Pin_16), X4.2 (Pin_2)
- net RAM_~{SS}: now also X2.15 (Pin_15)
- net RGB0: now also R11.1; no longer V6.3 (RK)
- net RGB1: now also R12.1; no longer V6.2 (GK)
- net RGB2: now also R13.1; no longer V6.1 (BK)
- net SPI_SCK: now also X3.15 (Pin_15), X4.9 (Pin_9)
- net SPI_SI: now also X3.14 (Pin_14), X4.7 (Pin_7)
- net SPI_SO: now also X3.13 (Pin_13), X4.8 (Pin_8)
- net SPI_~{HOLD}: now also X4.6 (Pin_6)
- net SPI_~{WP}: now also X4.5 (Pin_5)
- net USBD+: now also V2.6 (I/O1); no longer R2.1
- net USBD-: now also V2.4 (I/O2)
- net USB_P+: now also V1.43 (IOT_49a); no longer V1.4 (IOB_8a)
- net USB_P-: now also V1.42 (IOT_51a), R5.2; no longer V1.3 (IOB_9b)
- net VBUS: now also V2.5 (VBUS), X3.1 (Pin_1)
- net ~{CONF}_I: now also V1.3 (IOB_9b); no longer V1.42 (IOT_51a)
- net IOB_13b: now reaches V1.6 (IOB_13b)
- net IOB_13b: now also X3.6 (Pin_6)
- net IOT_45a: now reaches V1.37 (IOT_45a_G1)
- net IOT_45a: now also X2.11 (Pin_11)
- net IOB_18a: now reaches V1.10 (IOB_18a)
- net IOB_18a: now also X3.8 (Pin_8)
- net IOB_20a: now reaches V1.11 (IOB_20a)
- net IOB_20a: now also X3.9 (Pin_9)
- net IOB_24a: now reaches V1.13 (IOB_24a)
- net IOB_24a: now also X3.12 (Pin_12)
- net IOB_23b: now reaches V1.21 (IOB_23b)
- net IOB_23b: now also X3.11 (Pin_11)
- net IOB_16a: now reaches V1.9 (IOB_16a)
- net IOB_16a: now also X3.7 (Pin_7)
- net IOT_48b: now reaches V1.36 (IOT_48b)
- net IOT_48b: now also X3.4 (Pin_4)
- net IOT_41a: now reaches V1.28 (IOT_41a)
- net IOT_41a: now also X2.7 (Pin_7)
- net 1V2EN: now reaches C13.1, JP1.2 (B), V3.6 (VOUT1)
- net IOT_46b: now reaches V1.35 (IOT_46b_G0)
- net IOT_46b: now also X3.10 (Pin_10)
- net IOT_36b: now reaches V1.25 (IOT_36b)
- net IOT_36b: now also X2.3 (Pin_3)
- net IOT_38b: now reaches V1.27 (IOT_38b)
- net IOT_38b: now also X2.5 (Pin_5)
- net IOB_6a: now reaches V1.2 (IOB_6a)
- net IOB_6a: now also X3.5 (Pin_5)
- net IOB_3b: now reaches V1.44 (IOB_3b_G6)
- net IOB_3b: now also X3.2 (Pin_2)
- net USB_HS: now reaches V1.45 (IOB_5b)
- net USB_HS: now also R1.2
- net IOB_0a: now reaches V1.46 (IOB_0a)
- net IOB_0a: now also X2.13 (Pin_13)
- net IOB_2a: now reaches V1.47 (IOB_2a)
- net IOB_2a: now also X2.14 (Pin_14)
- net IOB_4a: now reaches V1.48 (IOB_4a)
- net IOB_4a: now also X3.3 (Pin_3)
- net IOT_42b: now reaches V1.31 (IOT_42b)
- net IOT_42b: now also X2.8 (Pin_8)
- net IOT_44b: now reaches V1.34 (IOT_44b)
- net IOT_44b: now also X2.10 (Pin_10)
- net IOT_37b: now reaches V1.23 (IOT_37a)
- net IOT_37b: now also X2.4 (Pin_4)
- net 3V3EN: now reaches C14.1, JP2.2 (B), V3.5 (VOUT2)
- net IOT_39a: now reaches V1.26 (IOT_39a)
- net IOT_39a: now also X2.6 (Pin_6)
- net IOT_43a: now reaches V1.32 (IOT_43a)
- net IOT_43a: now also X2.9 (Pin_9)
- new net IOB_8a: V1.4 (IOB_8a), X2.12 (Pin_12)
- new net RGB_B: R13.2, V6.1 (BK)
- new net RGB_G: R12.2, V6.2 (GK)
- new net RGB_R: R11.2, V6.3 (RK)
- new net USBDP+: R1.1, R2.1, V2.1 (I/O1)
- new net USBDP-: R5.1, V2.3 (I/O2)
- no-connect marks 4 -> 5
Other:
- note added: "3V3"
- note added: "Tag-Connect"
- note added: "symbol pin assignment reset !!!"
- note added: "yet2order!"
- note removed: "Testpoints"
- moved on the sheet: C1, C10, C11, C12, C13, C14, C16, C17, C18, C2, C5, C6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

Commit message: initial pcb layout
Parts:
- removed R6: 1Meg, Resistor_SMD:R_0402_1005Metric, symbol Device:R_Small
- removed X2, X3: Conn_01x16, Connector_PinHeader_2.54mm:PinHeader_1x16_P2.54mm_Vertical, symbol Connector_Generic:Conn_01x16
- added X2, X3: Conn_01x17, Connector_PinHeader_2.54mm:PinHeader_1x17_P2.54mm_Vertical, symbol Connector_Generic:Conn_01x17
- X4: footprint Connector:Tag-Connect_TC2050-IDC-NL_2x05_P1.27mm_Vertical -> Connector:Tag-Connect_TC2050-IDC-FP_2x05_P1.27mm_Vertical
- renumbered C16 to C1, C22 to C10, C13 to C11, C14 to C12, C5 to C13, C6 to C14, C7 to C15, C15 to C16, C8 to C17, C1 to C18, C9 to C19, C17 to C2, C10 to C20, C18 to C21, C2 to C22, C11 to C4, C4 to C5, C12 to C6, C19 to C7, C21 to C8, C20 to C9, R16 to R1, R5 to R10, R15 to R11, R19 to R12, R11 to R13, R12 to R14, R13 to R15, R9 to R16, R18 to R17, R14 to R18, R10 to R2, R17 to R3, R3 to R4, R4 to R5, R8 to R6, R1 to R8, R2 to R9, V5 to V1, V8 to V2, V2 to V4, V4 to V5, V1 to V6, V6 to V7, V7 to V8
Connections:
- net IOB_23b is gone; now on net RAM_~{SS}: V6.21 (IOB_23b)
- net +1V2: now also X2.2 (Pin_2)
- net +3V3: now also C16.1, X4.1 (Pin_1), X2.1 (Pin_1); no longer C16.2
- net CDONE: now also X4.10 (Pin_10)
- net FLASH_~{SS}: now also X4.2 (Pin_2), X3.17 (Pin_17); no longer X4.10 (Pin_10)
- net GND: now also C16.2, X1.S1 (SHIELD), X4.3 (Pin_3), X2.17 (Pin_17); no longer C16.1, X4.2 (Pin_2)
- net IOB_0a: now also X3.2 (Pin_2)
- net IOB_13b: now also X3.8 (Pin_8)
- net IOB_16a: now also X3.9 (Pin_9)
- net IOB_18a: now also X3.10 (Pin_10)
- net IOB_20a: now also X3.11 (Pin_11)
- net IOB_24a: now also X3.12 (Pin_12)
- net IOB_2a: now also X3.3 (Pin_3)
- net IOB_3b: now also X3.4 (Pin_4)
- net IOB_4a: now also X3.5 (Pin_5)
- net IOB_6a: now also X3.6 (Pin_6)
- net IOB_8a: now also X3.7 (Pin_7)
- net IOT_36b: now also X2.13 (Pin_13)
- net IOT_37b: now also X2.12 (Pin_12)
- net IOT_38b: now also X2.11 (Pin_11)
- net IOT_39a: now also X2.10 (Pin_10)
- net IOT_41a: now also X2.9 (Pin_9)
- net IOT_42b: now also X2.8 (Pin_8)
- net IOT_43a: now also X2.7 (Pin_7)
- net IOT_44b: now also X2.6 (Pin_6)
- net IOT_45a: now also X2.5 (Pin_5)
- net IOT_46b: now also X2.4 (Pin_4)
- net IOT_48b: now also X2.3 (Pin_3)
- net RAM_~{SS}: now also X4.7 (Pin_7), X3.13 (Pin_13); no longer V6.20 (IOB_25b_G3)
- net SPI_SCK: now also X4.4 (Pin_4), X3.15 (Pin_15); no longer X4.9 (Pin_9)
- net SPI_SI: now also X4.6 (Pin_6), X2.16 (Pin_16); no longer X4.7 (Pin_7)
- net SPI_SO: now also X3.14 (Pin_14)
- net SPI_~{HOLD}: now also V6.19 (IOB_29b), X4.9 (Pin_9), X3.16 (Pin_16); no longer V6.18 (IOB_31b), X4.6 (Pin_6)
- net SPI_~{WP}: now also V6.18 (IOB_31b), X2.15 (Pin_15); no longer V6.19 (IOB_29b)
- net VBUS: now also X3.1 (Pin_1)
- new net IOB_25b: V6.20 (IOB_25b_G3), X2.14 (Pin_14)
- no-connect marks 5 -> 2
Other:
- note removed: "3V3"
- moved on the sheet: C1, C10, C11, C12, C13, C14, C15, C16, C17, C18, C19, C2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
